File: Design Files/ECAD/HVHF_IIB/_autosave-HVHF_IIB.kicad_pcb (KiCad board)
At the start: 2 copper layers, 36 parts, among them J1 1984963, J2 1984963, Q1 PNP, Q2 BFP196E6327HTSA1, T1 BFU590G, T1 NPN

Commit message: adds footprints
Parts:
- added J3: CONSMA002-L, Library:LINX_CONSMA002-L, F.Cu at (-314.9, 57.0)
Connections:
- J1 pad 1: unconnected-(J1-Pad1) -> +VDC
- J1 pad 2: unconnected-(J1-Pad2) -> GND
- J2 pad 1: unconnected-(J2-Pad1) -> +5V
- J2 pad 2: unconnected-(J2-Pad2) -> GND
