File: Design Files/ECAD/HVHF_IIB/HVHF_IIB.kicad_pcb (KiCad board)
At the start: 4 copper layers, 117 x 79 mm, 64 parts, among them J1 1984963, J2 1984963, J3 731375003, J4 CONSMA002-L, Q1 PNP, Q2 BFP196E6327HTSA1, T1 BFU590G, T10 BFQ252, T11 BFQ252, T12 BFQ252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

Commit message: pcb work
routing
components
3d models
net classes
Parts:
- added D3: 1N5408, Diode_THT:D_DO-201AD_P15.24mm_Horizontal, F.Cu at (177.8, 85.0)
- added D4: 1N5408, Diode_THT:D_DO-201AD_P15.24mm_Horizontal, F.Cu at (123.0, 73.0)
- added F1: Fuse, Library:FUSE_4527, F.Cu at (183.0, 75.0)
- added F2: Fuse, Library:FUSE_4527, F.Cu at (133.0, 63.0)
- added J5: 1984963, 1_My_Custom_Library:CONN_1984963, F.Cu at (153.7, 61.0)
- added PCB1: ~EC1U, Library:PCB_EC1U, F.Cu at (150.0, 100.0)
- R12, R20, R21, R22: footprint Resistor_SMD:R_0805_2012Metric_Pad1.20x1.40mm_HandSolder -> Library:RES_3560_TEC
- moved R22 68.0 mm to (144.1, 136.5), turned to 90 degrees
- moved R19 66.3 mm to (136.9, 102.0), turned to -90 degrees
- moved J1 61.7 mm to (174.7, 61.0), turned to 180 degrees
- moved T12 60.7 mm to (142.2, 120.0), turned to 90 degrees
- moved J4 58.0 mm to (168.0, 139.0), turned to 0 degrees
- moved HS10 57.1 mm to (145.2, 120.0), turned to -90 degrees
- moved R21 55.8 mm to (159.1, 136.5), turned to 90 degrees
- moved C11 53.3 mm to (105.8, 112.6)
- moved R12 52.7 mm to (190.1, 136.9), turned to 90 degrees
- moved T9 52.6 mm to (142.2, 103.0), turned to 90 degrees
- moved C4 50.9 mm to (98.2, 102.2), turned to 180 degrees
- moved J2 49.5 mm to (113.7, 61.0), turned to 180 degrees
- moved HS9 48.4 mm to (145.2, 103.0), turned to -90 degrees
- moved C1 48.2 mm to (97.7, 120.9)
- moved R20 47.6 mm to (177.4, 136.7), turned to 90 degrees
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Connections:
- J1 pad 1: +VDC -> /+80V_IN
- J2 pad 1: +5V -> /+5V_IN
- T6 pad 2: Net-(T6-C) -> +VDC
- T7 pad 2: Net-(T6-C) -> +VDC
- T9 pad 2: Net-(T6-C) -> +VDC
Routing:
- net Net-(Q1-C): track 0.00 -> 23.7 mm
- net Net-(T1-C): track 0.00 -> 17.9 mm
- net Net-(D2-A): track 0.00 -> 12.3 mm
- net input: track 0.00 -> 11.1 mm
- net Net-(Q2-E): track 0.00 -> 11.1 mm, vias 0 -> 1
- net Net-(C1-Pad1): track 0.00 -> 3.97 mm
- net Net-(Q2-B): track 0.00 -> 3.92 mm
- net /FB2: track 0.00 -> 3.27 mm
Other:
- board size 117 x 79 mm -> 125 x 90 mm

Commit message: began routing
Parts:
- moved C5 49.4 mm to (111.3, 72.9)
- moved R11 17.9 mm to (137.8, 83.5), turned to -90 degrees
- moved Q1 17.2 mm to (104.6, 121.5), turned to 0 degrees
- moved C6 13.3 mm to (177.2, 83.4), turned to -90 degrees
- moved R10 11.6 mm to (108.0, 97.0), turned to -90 degrees
- moved R31 11.5 mm to (137.0, 123.5)
- moved D3 10.7 mm to (187.8, 88.8)
- moved C10 10.5 mm to (137.0, 117.5), turned to 90 degrees
- moved F1 10.1 mm to (190.9, 68.8), turned to 90 degrees
- moved R4 10.1 mm to (118.5, 125.2)
- moved D4 6.24 mm to (116.8, 73.0)
- moved R6 5.90 mm to (103.2, 109.6)
- moved R2 3.06 mm to (115.2, 123.8), turned to -90 degrees
- moved C2 2.75 mm to (112.4, 125.3)
- moved D2 2.75 mm to (109.2, 125.1)
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Routing:
- net /FB1: track 0.00 -> 58.8 mm
- net Net-(T12-B): track 0.00 -> 24.9 mm
- net Net-(T1-E): track 0.00 -> 21.1 mm
- net Net-(T8-B): track 0.00 -> 20.7 mm, vias 0 -> 1
- net Net-(D4-A): track 0.00 -> 20.1 mm
- net Net-(Q1-C): track 23.7 -> 6.80 mm
- net Net-(T2-B): track 0.00 -> 14.1 mm
- net +5V: track 0.00 -> 12.9 mm, vias 0 -> 5
- net Net-(D1-K): track 0.00 -> 12.4 mm
- net GND: track 0.00 -> 11.5 mm, vias 0 -> 8
- net Net-(Q2-E): track 11.1 -> 22.6 mm, vias 1 -> 0
- net /FB2: track 3.27 -> 13.8 mm
- net /+5V_IN: track 0.00 -> 8.12 mm
- net +VDC: track 0.00 -> 7.52 mm, vias 0 -> 2
- net Net-(T3-C): track 0.00 -> 6.38 mm
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
Commit message: pcb routing
routing
updated pcb brd footprint
Parts:
- moved LOGO1 42.5 mm to (150.0, 78.0)
- moved D3 17.9 mm to (205.5, 86.8), turned to 180 degrees
- moved R18 11.8 mm to (152.0, 99.2), turned to -90 degrees
- moved R17 11.8 mm to (168.0, 99.2)
- moved R3 11.8 mm to (183.0, 99.2)
- moved R10 9.53 mm to (114.5, 104.0), turned to 180 degrees
- moved R13 7.32 mm to (136.0, 104.2), turned to -90 degrees
- moved C4 5.54 mm to (96.2, 97.0)
- moved R8 3.68 mm to (97.0, 116.0)
- moved R19 2.91 mm to (136.0, 99.2)
- moved R9 2.69 mm to (105.5, 104.0), turned to 180 degrees
- moved R11 2.67 mm to (136.8, 86.0)
- moved R14 2.38 mm to (121.2, 101.5)
- moved R7 2.16 mm to (99.8, 115.9)
- moved R31 1.83 mm to (136.0, 122.0)
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Connections:
- net Net-(D3-A) renamed /F1
- net Net-(D4-A) renamed /F2
Routing:
- net Net-(R13-Pad1): track 3.02 -> 53.7 mm
- net output: track 0.00 -> 48.1 mm
- net Net-(T4-C): track 0.00 -> 33.2 mm
- net Net-(T10-C): track 0.00 -> 32.1 mm
- net Net-(T12-C): track 0.00 -> 31.9 mm
- net Net-(T11-C): track 0.00 -> 31.7 mm
- net Net-(T4-B): track 0.00 -> 27.3 mm
- net Net-(T10-B): track 0.00 -> 27.0 mm
- net Net-(T11-B): track 0.00 -> 26.3 mm
- net /F2: track 20.1 -> 0.00 mm
- net GND: track 11.5 -> 26.2 mm, vias 8 -> 12
- net Net-(Q2-E): track 22.6 -> 32.7 mm, vias 0 -> 2
- net /+5V_IN: track 8.12 -> 0.00 mm
- net +5V: track 12.9 -> 7.78 mm
- net /FB1: track 58.8 -> 53.8 mm
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- added copper zone on F.Cu, net +5V
- added copper zone on F.Cu, net /+5V_IN
- added copper zone on F.Cu, net /+80V_IN
- added copper zone on F.Cu, net /F1
- added copper zone on F.Cu, net /F2

Commit message: routing
Did DRC
Did ERC (some errors to fix)
Parts:
- LOGO1: footprint Library:Bard_Logo -> Library:LOGO_M
- moved LOGO1 8.31 mm to (149.0, 69.8)
- moved J3 0.75 mm to (112.2, 129.8)
- moved T2 0.26 mm to (125.5, 119.5)
- moved T10 0.21 mm to (172.8, 119.5)
- moved T4 0.21 mm to (187.8, 119.5)
- moved T5 0.21 mm to (187.8, 102.5)
- moved T6 0.21 mm to (172.8, 102.5)
- moved HS3 0.21 mm to (190.8, 119.5)
- moved HS4 0.21 mm to (190.8, 102.5)
- moved HS5 0.21 mm to (175.8, 102.5)
- moved HS6 0.21 mm to (175.8, 119.5)
- moved T3 0.21 mm to (125.5, 102.5)
- moved HS1 0.17 mm to (128.3, 119.5)
- moved T11 0.06 mm to (156.5, 119.5)
- moved T12 0.06 mm to (141.5, 119.5)
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Routing:
- net GND: track 26.2 -> 11.8 mm, vias 12 -> 10
Other:
- board text added: "Physics Lab HVHF-IIB-01"
