File: Design Files/ECAD/HVHF_IIB/HVHF_IIB.kicad_sch (KiCad schematic)
At the start: 70 parts, among them J1 1984963, J2 1984963, J3 731375003, J4 CONSMA002-L, J5 1984963, Q1 PNP, Q2 BFP196E6327HTSA1, T1 BFU590G, T10 BFQ252, T11 BFQ252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

Commit message: routing
Did DRC
Did ERC (some errors to fix)
Parts:
- LOGO1: footprint Library:Bard_Logo -> Library:LOGO_M
Connections:
- net GND: no longer PCB1.1 (GND_SCREW)
Changed lines of the file:
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@@
+    (stroke (width 0) (type default))
+  )
+  (wire (pts (xy 262.89 142.24) (xy 265.43 142.24))
+    (stroke (width 0) (type default))
+  )
+  (wire (pts (xy 228.6 142.24) (xy 228.6 144.78))
+    (stroke (width 0) (type default))
+  )
+  (wire (pts (xy 110.49 133.35) (xy 111.76 133.35))
+    (stroke (width 0) (type default))
+  )
+  (wire (pts (xy 250.19 114.3) (xy 250.19 124.46))
+    (stroke (width 0) (type default))
+  )
+  (wire (pts (xy 76.2 38.1) (xy 77.47 38.1))
+    (stroke (width 0) (type default))
+  )
+  (wire (pts (xy 151.13 133.35) (xy 156.21 133.35))
+    (stroke (width 0) (type default))
+  )
+  (wire (pts (xy 231.14 41.91) (xy 231.14 44.45))
+    (stroke (width 0) (type default))
+  )
+  (wire (pts (xy 62.23 166.37) (xy 62.23 162.56))
+    (stroke (width 0) (type default))
+  )
+  (wire (pts (xy 119.38 125.73) (xy 119.38 128.27))
+    (stroke (width 0) (type default))
+  )
+  (wire (pts (xy 115.57 156.21) (xy 115.57 158.75))
+    (stroke (width 0) (type default))
+  )
+  (wire (pts (xy 163.83 140.97) (xy 165.1 140.97))
+    (stroke (width 0) (type default))
+  )
+  (wire (pts (xy 184.15 114.3) (xy 184.15 123.19))
+    (stroke (width 0) (type default))
+  )
+  (wire (pts (xy 100.33 148.59) (xy 111.76 148.59))
+    (stroke (width 0) (type default))
+  )
+  (wire (pts (xy 115.57 166.37) (xy 115.57 186.69))
+    (stroke (width 0) (type default))
+  )
+  (wire (pts (xy 151.13 114.3) (xy 184.15 114.3))
+    (stroke (width 0) (type default))
+  )
+  (wire (pts (xy 72.39 133.35) (xy 72.39 135.89))
+    (stroke (width 0) (type default))
+  )
+  (wire (pts (xy 119.38 114.3) (xy 138.43 114.3))
+    (stroke (width 0) (type default))
+  )
+  (wire (pts (xy 48.26 38.1) (xy 50.8 38.1))
     (stroke (width 0) (type default))
   )
@@
     (stroke (width 0) (type default))
   )
-  (wire (pts (xy 262.89 142.24) (xy 265.43 142.24))
-    (stroke (width 0) (type default))
-  )
-  (wire (pts (xy 228.6 142.24) (xy 228.6 144.78))
-    (stroke (width 0) (type default))
-  )
-  (wire (pts (xy 110.49 133.35) (xy 111.76 133.35))
-    (stroke (width 0) (type default))
-  )
-  (wire (pts (xy 250.19 114.3) (xy 250.19 124.46))
-    (stroke (width 0) (type default))
-  )
-  (wire (pts (xy 76.2 38.1) (xy 77.47 38.1))
-    (stroke (width 0) (type default))
-  )
-  (wire (pts (xy 151.13 133.35) (xy 156.21 133.35))
-    (stroke (width 0) (type default))
-  )
-  (wire (pts (xy 231.14 41.91) (xy 231.14 44.45))
-    (stroke (width 0) (type default))
-  )
-  (wire (pts (xy 62.23 166.37) (xy 62.23 162.56))
-    (stroke (width 0) (type default))
-  )
-  (wire (pts (xy 119.38 125.73) (xy 119.38 128.27))
-    (stroke (width 0) (type default))
-  )
-  (wire (pts (xy 115.57 156.21) (xy 115.57 158.75))
-    (stroke (width 0) (type default))
-  )
-  (wire (pts (xy 163.83 140.97) (xy 165.1 140.97))
-    (stroke (width 0) (type default))
-  )
-  (wire (pts (xy 184.15 114.3) (xy 184.15 123.19))
-    (stroke (width 0) (type default))
-  )
-  (wire (pts (xy 100.33 148.59) (xy 111.76 148.59))
-    (stroke (width 0) (type default))
-  )
-  (wire (pts (xy 115.57 166.37) (xy 115.57 186.69))
-    (stroke (width 0) (type default))
-  )
-  (wire (pts (xy 151.13 114.3) (xy 184.15 114.3))
-    (stroke (width 0) (type default))
-  )
-  (wire (pts (xy 72.39 133.35) (xy 72.39 135.89))
-    (stroke (width 0) (type default))
-  )
-  (wire (pts (xy 119.38 114.3) (xy 138.43 114.3))
-    (stroke (width 0) (type default))
-  )
-  (wire (pts (xy 48.26 38.1) (xy 50.8 38.1))
-    (stroke (width 0) (type default))
-  )
   (wire (pts (xy 85.09 133.35) (xy 100.33 133.35))
     (stroke (width 0) (type default))
@@
     (stroke (width 0) (type default))
   )
+  (wire (pts (xy 184.15 133.35) (xy 184.15 148.59))
+    (stroke (width 0) (type default))
+  )
+  (wire (pts (xy 102.87 40.64) (xy 97.79 40.64))
+    (stroke (width 0) (type default))
+  )
+  (wire (pts (xy 119.38 81.28) (xy 119.38 87.63))
+    (stroke (width 0) (type default))
+  )
+  (wire (pts (xy 72.39 185.42) (xy 72.39 186.69))
+    (stroke (width 0) (type default))
+  )
+  (wire (pts (xy 76.2 38.1) (xy 76.2 43.18))
+    (stroke (width 0) (type default))
+  )
+  (wire (pts (xy 80.01 148.59) (xy 92.71 148.59))
+    (stroke (width 0) (type default))
+  )
   (wire (pts (xy 63.5 81.28) (xy 106.68 81.28))
     (stroke (width 0) (type default))
   )
-  (wire (pts (xy 184.15 133.35) (xy 184.15 148.59))
-    (stroke (width 0) (type default))
-  )
-  (wire (pts (xy 102.87 40.64) (xy 97.79 40.64))
-    (stroke (width 0) (type default))
-  )
-  (wire (pts (xy 119.38 81.28) (xy 119.38 87.63))
-    (stroke (width 0) (type default))
-  )
-  (wire (pts (xy 72.39 185.42) (xy 72.39 186.69))
-    (stroke (width 0) (type default))
-  )
-  (wire (pts (xy 76.2 38.1) (xy 76.2 43.18))
-    (stroke (width 0) (type default))
-  )
-  (wire (pts (xy 80.01 148.59) (xy 92.71 148.59))
-    (stroke (width 0) (type default))
-  )
   (wire (pts (xy 220.98 149.86) (xy 215.9 149.86))
     (stroke (width 0) (type default))
@@
     (stroke (width 0) (type default))
   )
-  (wire (pts (xy 118.11 31.75) (xy 118.11 27.94))
-    (stroke (width 0) (type default))
-  )
   (wire (pts (xy 43.18 133.35) (xy 43.18 135.89))
     (stroke (width 0) (type default))
@@
   )
   (wire (pts (xy 76.2 35.56) (xy 76.2 38.1))
-    (stroke (width 0) (type default))
-  )
-  (wire (pts (xy 118.11 27.94) (xy 120.65 27.94))
     (stroke (width 0) (type default))
   )
@@
     )
   )
-  (symbol (lib_id "power:GND") (at 118.11 31.75 0) (unit 1)
-    (in_bom yes) (on_board yes) (dnp no) (fields_autoplaced)
-    (property "Reference" "#PWR027" (at 118.11 38.1 0)
-      (effects (font (size 1.27 1.27)) hide)
-    )
-    (property "Value" "GND" (at 118.11 36.83 0)
-      (effects (font (size 1.27 1.27)))
-    )
-    (property "Footprint" "" (at 118.11 31.75 0)
-      (effects (font (size 1.27 1.27)) hide)
-    )
-    (property "Datasheet" "" (at 118.11 31.75 0)
-      (effects (font (size 1.27 1.27)) hide)
-    )
-    (pin "1")
-    (instances
-      (project "HVHF_IIB"
-        (path "/a4785c7b-64d4-4462-915b-801e602c6997"
-          (reference "#PWR027") (unit 1)
-        )
-      )
-    )
-  )
   (symbol (lib_id "Device:R") (at 234.95 142.24 270) (unit 1)
     (in_bom yes) (on_board yes) (dnp no)
@@
       (effects (font (size 1.27 1.27)) hide)
     )
-    (pin "1")
     (instances
       (project "HVHF_IIB"
@@
       (effects (font (size 1.27 1.27)))
     )
-    (property "Footprint" "Library:Bard_Logo" (at 193.04 62.23 0)
-      (effects (font (size 1.27 1.27)) hide)
-    )
+    (property "Footprint" "Library:LOGO_M" (at 193.04 62.23 0)
+      (effects (font (size 1.27 1.27)) hide)
+    )
